File: v6/PROJET_KICAD/SUPPLY_CENTIPEDE.kicad_sch (KiCad schematic)
At the start: 26 parts, among them IC1 MCP73871-2CCI_ML, IC2 TPS61090RSAR, J1 USB4110-GF-A, J2 S2B-PH-SM4-TB_LF__SN_

Commit message: Correct errors on supply schematic
Parts:
- C2: value (none) -> 2.2uF
- C6: value (none) -> 100uF
- L1: value (none) -> 6.8uH
- Q1: value (none) -> PBSS301PZ; footprint (none) -> Package_TO_SOT_SMD:SOT-223-3_TabPin2
Connections:
- net GND: now also R4.1; no longer IC1.5 (THERM), R4.2
- net VLIPO: now also J2.2
- net 5V: now reaches C2.1, C6.1, IC2.1 (VOUT_1), IC2.15 (VOUT_2), IC2.16 (VOUT_3), R3.1, R5.1
- net 5V: no longer J2.2
- net at IC2.14 (FB), R3.2: now also R4.2; no longer R4.1
- net VUSBC renamed VBUS
Other:
- moved on the sheet: C1, C2, C4, C6, C7, D1, D2, J2, L1, Q1, R1, R2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
